File: Microrat.kicad_pcb (KiCad board)
At the start: 2 copper layers, 80 x 109 mm, 32 parts, among them J1 Conn_01x03_Socket, J2 Conn_01x03_Socket, J3 Conn_01x02_Pin, J4 Conn_01x02_Pin, J5 Conn_01x05_Pin, J6 Conn_01x02_Pin, J7 Conn_01x05_Pin, J8 Conn_01x05_Pin, SW1 SW_DPDT_x2, SW2 SW_MEC_5E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

Commit message: Final Heute
Parts:
- SW1: footprint Button_Switch_THT:SW_E-Switch_EG1271_SPDT -> Library:Wippschalter
- moved D3 6.08 mm to (254.0, 203.0)
- moved R2 6.08 mm to (258.1, 202.9)
- moved SW1 5.60 mm to (250.0, 218.0)
- moved SW2 2.00 mm to (265.8, 195.8)
Connections:
- SW1 pad 1: Batt_out -> (no net)
- SW1 pad 2: +BATT -> (no net)
- SW1 pad 3: unconnected-(SW1A-C-Pad3) -> (no net)
