File: Microrat.kicad_sch (KiCad schematic)
At the start: 24 parts, among them J1 Conn_01x03_Socket, J2 Conn_01x03_Socket, M1 Motor_DC, M2 Motor_DC, SW1 SW_DPDT_x2, U1 L293D, U10 L7806, U2 LD1117S50TR_SOT223, U4 HC-SR04, U8 GP2Y0A51SK0F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

Commit message: Schematic aktuell
Connections:
- net +BATT: now also SW1.2 (B); no longer C1.1, C3.1, U10.1 (IN), U2.3 (VI)
- net Batt_out: now reaches SW1.1 (A)
- net Batt_out: now also C1.1, C3.1, U10.1 (IN), U2.3 (VI)
Other:
- moved on the sheet: C1, C2, D1, D2, D3, J1, J2, R1, R2, R3, SW1A, U2

Commit message: neue Schematic
Parts:
- removed U8, U9: GP2Y0A51SK0F, GP2Y0A21YK0F:22-23-2031, symbol GP2Y0A51SK0F:GP2Y0A21YK0F
- added C5: C100nF, symbol Device:C
- added J3: Conn_01x02_Pin, Connector_Wire:SolderWire-2.5sqmm_1x02_P7.2mm_D2.4mm_OD3.6mm, symbol Connector:Conn_01x02_Pin
- added J4: Conn_01x02_Pin, Connector_PinHeader_1.00mm:PinHeader_1x02_P1.00mm_Vertical, symbol Connector:Conn_01x02_Pin
- added J5: Conn_01x05_Pin, Connector_PinHeader_1.00mm:PinHeader_1x05_P1.00mm_Vertical, symbol Connector:Conn_01x05_Pin
- added SW2: SW_MEC_5E, Button_Switch_SMD:SW_MEC_5GSH9, symbol Switch:SW_MEC_5E
- R1, R3: value R -> R128
- R2: value R -> R68
- U3: footprint (none) -> XMC1402T038X0128AAXUMA1:SOP50P640X120-38N
Connections:
- net +3.3V is gone; now on net +5V: U5.3 (VCC), U6.3 (VCC)
- net +5V: now also U3.10 (VDD,VDDP), C5.2, SW2.3 (K), SW2.4 (A)
- net +BATT: now also J3.2 (Pin_2)
- net Freedig1: now also J5.1 (Pin_1)
- net Freedig2: now also J5.2 (Pin_2)
- net Freedig3: now also J5.3 (Pin_3)
- net Freedig4: now also J5.4 (Pin_4)
- net Freedig5: now also J5.5 (Pin_5)
- net GND: now also U3.9 (VSS,VSSP), C5.1, J3.1 (Pin_1)
- net UART_RX: now also J4.1 (Pin_1)
- net UART_TX: now also J4.2 (Pin_2)
- new net Switch: SW2.1, SW2.2
- no-connect marks 0 -> 16
Other:
- note added: "Conn_Batt"
- note added: "Conn_IO"
- note added: "Conn_RxTx"
- note added: "Switch_User"
- note removed: "Infra 1"
- note removed: "Infra 2"
- note removed: "Infrarot Sensoren"
- moved on the sheet: J1, J2, U3

Commit message: XMC neue Flags
Connections:
- net CAP: now also U3.31 (P0.12); no longer U3.19 (P0.2)
- net Freedig1: now also U3.5 (P2.8); no longer U3.32 (P0.13)
- net Freedig2: now also U3.4 (P2.7); no longer U3.31 (P0.12)
- net Freedig3: now also U3.3 (P2.6); no longer U3.30 (P0.11)
- net Freedig4: now also U3.2 (P2.5); no longer U3.29 (P0.10)
- net Freedig5: now also U3.1 (P2.4); no longer U3.28 (P0.9)
- net Infra_out1: now also U3.36 (P2.1); no longer U3.38 (P2.3)
- net Input 1: now also U3.11 (P1.5); no longer U3.1 (P2.4)
- net Input 2: now also U3.12 (P1.4); no longer U3.2 (P2.5)
- net Input 3: now also U3.13 (P1.3); no longer U3.3 (P2.6)
- net Input 4: now also U3.14 (P1.2); no longer U3.4 (P2.7)
- net M1 A: now also U3.22 (P0.5); no longer U3.16 (P1.0)
- net M1 B: no longer U3.15 (P1.1)
- net M2 A: now also U3.21 (P0.4); no longer U3.14 (P1.2)
- net M2 B: no longer U3.13 (P1.3)
- net PWM 1: now also U3.15 (P1.1); no longer U3.20 (P0.3)
- net PWM 2: now also U3.16 (P1.0); no longer U3.21 (P0.4)
- net PWM 3: now also U3.8 (P2.11); no longer U3.22 (P0.5)
- net UART_RX: now also U3.24 (P0.7); no longer U3.37 (P2.2)
- net UART_TX: now also U3.23 (P0.6); no longer U3.36 (P2.1)
- new net I2C_SCL: U3.19 (P0.2)
- new net I2C_SDA: U3.20 (P0.3)

Commit message: neuste Änderungen
Parts:
- added J6: Conn_01x02_Pin, Connector_PinHeader_1.00mm:PinHeader_1x02_P1.00mm_Vertical, symbol Connector:Conn_01x02_Pin
Connections:
- net IO is gone; now on net CAP: U4.3 (ECHO)
- net Auge 1: now also U3.6 (P2.9)
- net Auge 2: now also U3.7 (P2.10)
- net I2C_SCL: now also J6.2 (Pin_2)
- net I2C_SDA: now also J6.1 (Pin_1)
- net M1 B: no longer names the net of U5.5 (B)
- net M2 B: no longer names the net of U6.5 (B)
Other:
- note added: "Conn_I2C"
- moved on the sheet: J1, J2, SW2

Commit message: Debug
Parts:
- added U7: ~, symbol XMC_Debug:Debug_Stecker
Other:
- note added: "Debug Stecker"
Changed lines of the file:
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@@
+	)
+	(rectangle
+		(start 66.04 130.81)
+		(end 100.33 151.13)
+		(stroke
+			(width 0.254)
+			(type dash)
+		)
+		(fill
+			(type none)
+		)
 	)
 	(rectangle
@@
 		)
 	)
+	(text "Debug Stecker"
+		(exclude_from_sim no)
+		(at 83.82 128.778 0)
+		(effects
+			(font
+				(size 1.27 1.27)
+			)
+		)
+	)
 	(text "Magnetic Encoder M1"
 		(exclude_from_sim no)
@@
 					(unit 1)
 				)
+			)
+		)
+	)
+	(symbol
+		(lib_id "XMC_Debug:Debug_Stecker")
+		(at 83.82 134.62 0)
+		(unit 1)
+		(exclude_from_sim no)
+		(in_bom yes)
+		(on_board yes)
+		(dnp no)
+		(fields_autoplaced yes)
+		(property "Reference" "U7"
+			(at 83.185 133.35 0)
+			(effects
+				(font
+					(size 1.27 1.27)
+				)
+			)
+		)
+		(property "Value" "~"
+			(at 83.185 135.89 0)
+			(effects
+				(font
+					(size 1.27 1.27)
+				)
+			)
+		)
+		(property "Footprint" ""
+			(at 83.82 134.62 0)
+			(effects
+				(font
+					(size 1.27 1.27)
+				)
+				(hide yes)
+			)
+		)
+		(property "Datasheet" ""
+			(at 83.82 134.62 0)
+			(effects
+				(font
+					(size 1.27 1.27)
+				)
+				(hide yes)
+			)
+		)
+		(property "Description" ""
+			(at 83.82 134.62 0)
+			(effects
+				(font
+					(size 1.27 1.27)
+				)
+				(hide yes)
+			)
+		)
+		(pin "2"
+		)
+		(pin "7"
+		)
+		(pin "4"
+		)
+		(pin "3"
+		)
+		(pin "5"
+		)
+		(pin "7"
+		)
+		(pin "8"
+		)
+		(pin "1"
+		)
+		(instances
+			(project "Microrat"
+				(path "/aa0a1eb8-88c0-4621-81d3-41407e330c9d"
+					(reference "U7")
+					(unit 1)
+				)

Commit message: neue Änderungen
Parts:
- removed M1, M2: Motor_DC, symbol Motor:Motor_DC
- removed U5, U6: ~, symbol New_Library:Magnetic_Encoder_1
- added J7, J8: Conn_01x05_Pin, Connector_Wire:SolderWire-0.1sqmm_1x05_P3.6mm_D0.4mm_OD1mm, symbol Connector:Conn_01x05_Pin
- C1, C2, C3, C4, C5: footprint (none) -> Capacitor_SMD:C_0201_0603Metric
- D1, D2: footprint (none) -> LED_THT:LED_D3.0mm_Horizontal_O1.27mm_Z2.0mm
- R1, R2, R3: footprint (none) -> Resistor_SMD:R_0201_0603Metric
- SW1: footprint Button_Switch_SMD:SW_DPDT_CK_JS202011JCQN -> Button_Switch_THT:SW_CK_JS202011CQN_DPDT_Straight
- SW2: footprint Button_Switch_SMD:SW_MEC_5GSH9 -> Button_Switch_THT:SW_MEC_5GTH9
- U7: footprint (none) -> Connector_JST:JST_ACH_BM04B-ACHSS-A-GAN-ETF_1x04-1MP_P1.20mm_Vertical
Connections:
- net +5V: now also J7.3 (Pin_3), J8.3 (Pin_3)
- net GND: now also J7.5 (Pin_5), J8.5 (Pin_5)
- net M1 A: now also J7.4 (Pin_4)
- net M1 Enc: now also J7.1 (Pin_1)
- net M2 A: now also J8.4 (Pin_4)
- net M2 Enc: now also J7.2 (Pin_2)
- net M3 Enc: now also J8.1 (Pin_1)
- net M4 Enc: now also J8.2 (Pin_2)
- no-connect marks 16 -> 18
Other:
- note added: "????????????????????????"

Commit message: Final Heute
Parts:
- SW1: footprint Button_Switch_THT:SW_CK_JS202011CQN_DPDT_Straight -> Library:Wippschalter
- SW2: footprint Button_Switch_THT:SW_MEC_5GTH9 -> Button_Switch_THT:SW_PUSH_6mm_H4.3mm
Changed lines of the file:
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@@
 			)
 		)
-		(property "Footprint" "Button_Switch_THT:SW_MEC_5GTH9"
+		(property "Footprint" "Button_Switch_THT:SW_PUSH_6mm_H4.3mm"
 			(at 34.29 92.71 0)
 			(effects
@@
 			)
 		)
-		(property "Footprint" "Button_Switch_THT:SW_CK_JS202011CQN_DPDT_Straight"
+		(property "Footprint" "Library:Wippschalter"
 			(at 209.55 114.3 0)
 			(effects
